Commit message: add ok robot manip

File: src/home_robot/home_robot/agent/multitask/ok_robot_hw/hab_stretch/urdf/planner_calibrated_simplified.urdf (robot description, URDF)
Before this commit: robot stretch_description, 48 links, 47 joints
Links:
- removed link fake_link_x
- added link base_imu, mass 0.000901473198307758; collision mesh filename=../meshes/base_imu.STL; visual mesh filename=../meshes/base_imu.STL
- link base_link: mass 1.1912 -> 10.0723782659782; geometry collision box size=0.143197 0.324688 0.361202; visual mesh filename=../meshes/base_link.STL
- link camera_link: geometry collision box size=0.02505 0.09 0.025; visual mesh filename=../meshes/realsense2/d435.dae
- link caster_link: geometry visual mesh filename=../meshes/omni_wheel_m.STL
- link laser: geometry collision box size=0.0195 0.06994 0.06994; visual mesh filename=../meshes/laser.STL
- link link_arm_l0: mass 0.085003260946398 -> 0.101241250325294; geometry collision box size=0.059285 0.127573 0.2265; visual mesh filename=../meshes/link_arm_l0.STL
- link link_arm_l1: mass 0.051382 -> 0.0511763619538321; geometry collision box size=0.04725 0.04725 0.2265; visual mesh filename=../meshes/link_arm_l1.STL
- link link_arm_l2: mass 0.0571386353275368 -> 0.0569074368576238; geometry collision box size=0.05125 0.05125 0.2265; visual mesh filename=../meshes/link_arm_l2.STL
- link link_arm_l3: mass 0.0628927381893134 -> 0.0626921047058405; geometry collision box size=0.05525 0.05525 0.2265; visual mesh filename=../meshes/link_arm_l3.STL
- link link_arm_l4: mass 0.068095 -> 0.0676525455789735; geometry collision box size=0.05925 0.05925 0.2225; visual mesh filename=../meshes/link_arm_l4.STL
- link link_aruco_inner_wrist: geometry visual mesh filename=../meshes/link_aruco_inner_wrist.STL
- link link_aruco_left_base: geometry visual mesh filename=../meshes/link_aruco_left_base.STL
- link link_aruco_right_base: geometry visual mesh filename=../meshes/link_aruco_right_base.STL
- link link_aruco_shoulder: geometry visual mesh filename=../meshes/link_aruco_shoulder.STL
- link link_gripper_finger_left: geometry collision box size=0.013 0.03021 0.196835; visual mesh filename=../meshes/link_gripper_finger_left.STL
- link link_gripper_finger_right: geometry collision box size=0.013 0.03021 0.196835; visual mesh filename=../meshes/link_gripper_finger_right.STL
- link link_head: mass 0.133027236718691 -> 0.129454717596498; geometry collision box size=0.056453 0.131612 0.19515; visual mesh filename=../meshes/link_head.STL
- link link_head_pan: mass 0.0273764496535409 -> 0.035858341182617; geometry collision box size=0.043969 0.048193 0.122235; visual mesh filename=../meshes/link_head_pan.STL
- link link_head_tilt: mass 0.090217113313934 -> 0.0701242408063442; geometry collision box size=0.061014 0.068029 0.120844; visual mesh filename=../meshes/link_head_tilt.STL
- link link_left_wheel: mass 0.0042721 -> 0.01; geometry visual mesh filename=../meshes/link_left_wheel.STL
- link link_lift: mass 0.27218 -> 0.444820831236007; geometry collision box size=0.120261 0.137963 0.258855; visual mesh filename=../meshes/link_lift.STL
- link link_mast: mass 1.8285 -> 0.749143203376401; geometry collision box size=0.038125 0.038125 1.285; visual mesh filename=../meshes/link_mast.STL
- link link_right_wheel: mass 0.0042721 -> 0.01; geometry visual mesh filename=../meshes/link_right_wheel.STL
- link link_straight_gripper: geometry collision box size=0.052858 0.056076 0.108538; visual mesh filename=../meshes/link_straight_gripper.STL
- link link_wrist_pitch: geometry collision box size=0.043138 0.053359 0.064888; visual mesh filename=../meshes/link_wrist_pitch.STL
- link link_wrist_roll: geometry collision box size=0.0155 0.028888 0.028987; visual mesh filename=../meshes/link_wrist_roll.STL
- link link_wrist_yaw: mass 0.0404746907425003 -> 0.0405398981326229; geometry collision box size=0.029951 0.029976 0.038; visual mesh filename=../meshes/link_wrist_yaw.STL
- link link_wrist_yaw_bottom: geometry collision box size=0.0415 0.062919 0.0943; visual mesh filename=../meshes/link_wrist_yaw_bottom.STL
- link respeaker_base: mass 0.015643 -> 0.00969129410417277; geometry collision box size=0.042669 0.070906 0.079812; visual mesh filename=../meshes/link_respeaker.STL
Joints:
- removed joint joint_fake
- added joint joint_base_imu: type fixed, parent base_link, child base_imu, origin xyz=-0.12838 0.0031592 0.1474 rpy=-3.1416 0 -1.5708, axis 0 0 0
- joint base_theta_joint: limit (none) -> lower=0.0 upper=0.0 effort=100.0 velocity=1.0; origin xyz=0.0 0.0 0.0 rpy=0.0 0.0 0.0 -> xyz=0.0 0.0 0.0 rpy=0.0 0.0 -1.57079632679496
- joint base_y_joint: limit (none) -> lower=0.0 upper=0.0 effort=100.0 velocity=3.0; origin xyz=0 0 0 rpy=0.0 0.0 0.0 -> xyz=0 0 0 rpy=0.0 0.0 1.57079632679496
- joint camera_joint: origin xyz=0.02802960503838624 -0.007608222297947431 0.018218494141479257 rpy=0.010658876360659654 -0.0022761048951753793 0.018675317090921212 -> xyz=0.025070381118864622 -0.012287278361953074 0.017905872362600883 rpy=0.0027184810411859444 0.001558563349419062 -0.04777120277132254
- joint joint_arm_l0: origin xyz=0.0 0.0 -0.0137499999991968 rpy=7.63746778746202e-30 -3.80121128864402e-15 2.62707547767438e-15 -> xyz=0.0 0.0 -0.0137499999999938 rpy=-3.05317390622457e-16 -4.23236224076729e-16 -2.68425135229209e-17
- joint joint_arm_l1: origin xyz=0.0 0.0 0.0129999999999981 rpy=-7.63746778746202e-30 -7.88860905221012e-31 1.11022302462516e-16 -> xyz=0.0 0.0 0.013 rpy=7.41596560408007e-17 1.33876788296791e-16 -2.44545873596083e-16
- joint joint_arm_l2: origin xyz=0.0 0.0 0.013 rpy=0.0 1.57655765344625e-30 -1.66533453693773e-16 -> xyz=0.0 0.0 0.013 rpy=2.91385731014123e-16 4.44300759504684e-17 3.25691080516352e-16
- joint joint_arm_l3: origin xyz=0.0 0.0 0.013 rpy=7.68831233799385e-30 2.36716479416092e-30 2.29652732251143e-17 -> xyz=0.0 0.0 0.013 rpy=3.5742e-16 3.2123e-16 -2.4565e-16
- joint joint_arm_l4: origin xyz=-0.25956015433181046 -0.0059261537843136765 -0.005557384627505743 rpy=1.5619286973774569 -0.006924580188019336 -1.575847166561953 -> xyz=-0.25669443874094205 0.005713417002918588 0.0012296937814473496 rpy=1.5781652616599324 0.04551858006017695 -1.6181874684011688
- joint joint_aruco_right_base: origin xyz=-0.0015028 -0.1304972 0.1597482 rpy=0.0 0.0 -1.5707963267949 -> xyz=-0.00500000000000014 -0.1304972 0.1597482 rpy=0.0 0.0 -1.5707963267949
- joint joint_head: origin xyz=0.0 1.33 0.0 rpy=1.5707963267949 -1.5707963267949 3.1416 -> xyz=0.0 1.33 0.0 rpy=1.5708 -1.5615 3.1416
- joint joint_head_pan: origin xyz=0.1284513021260868 0.07637128403435504 0.00023722543808071166 rpy=-0.013467967166369273 0.005690738105448956 1.6024957766579377 -> xyz=0.14394738959044898 0.0689269242761915 -0.003064182445303723 rpy=0.008083283195200545 0.000583944763831834 1.620778470351339
- joint joint_head_tilt: origin xyz=0.0032337815907659225 0.030910701770693223 -0.04783143162927699 rpy=1.5763332066189244 -0.029319157204454882 -0.005080558641851002 -> xyz=-0.0038009318349181698 0.027661869381952295 -0.06046636278717248 rpy=1.583686486584009 0.038258710433179965 0.07682454066916562
- joint joint_laser: origin xyz=0.004 0.0 0.1664 rpy=0.0 0.0 3.1416 -> xyz=0.000502800000000914 0.0 0.1664 rpy=0.0 0.0 -3.14159265358979
- joint joint_left_wheel: origin xyz=0.0 0.17035 0.0508 rpy=-1.5708 2.6317e-16 -8.2057e-19 -> xyz=-0.00300000000001899 0.15765 0.0507999999999994 rpy=-1.5707963267949 3.16227047920818e-31 7.88745438253713e-16
- joint joint_lift: origin xyz=-0.037385 0.1666 0.0 rpy=-1.5708 1.5708 0.0 -> xyz=-0.0369217062323472 0.165471199999996 -0.000341653286793524 rpy=-1.57079632679552 1.5615431375292 -6.2942004366467e-13
- joint joint_mast: origin xyz=-0.07174416574437388 0.13780491000396983 0.03663931715774088 rpy=1.5780076046568878 0.016499709009588637 -0.007971437955302632 -> xyz=-0.06949477028757628 0.13838980304778414 0.027045430913364362 rpy=1.5646590837134537 -0.017304958691331196 0.04825274364916361; parent fake_link_x -> base_link
- joint joint_respeaker: origin xyz=0.0 1.37236408874452 0.00303065898329655 rpy=-1.5707963267949 -0.698131700797725 4.93295812652799e-16 -> xyz=1.09074743137871e-05 1.36992 0.00303572796911382 rpy=1.57079632679553 0.0 3.14159265358916
- joint joint_right_wheel: origin xyz=0.0 -0.17035 0.0508 rpy=-1.5708 1.2717e-16 4.8006e-17 -> xyz=-0.00300000000000034 -0.15765 0.0508000000000004 rpy=-1.57079632679489 -1.11022302462516e-16 7.28583859910277e-17
- joint joint_wrist_yaw: origin xyz=0.0830000000000654 -0.0307500000000129 0.0 rpy=1.5708 4.2595e-14 2.6415e-15 -> xyz=0.083 -0.03075 0.0 rpy=1.5708 4.2595e-14 2.6415e-15

File: src/home_robot/home_robot/agent/multitask/ok_robot_hw/hab_stretch/urdf/stretch_manip_mode.urdf (robot description, URDF)
Before this commit: robot stretch_description, 48 links, 47 joints
Links:
- removed link base_theta_link
- removed link base_xy_link
- removed link world
- added link base_imu, mass 0.00092; collision mesh filename=package://stretch_description/meshes/base_imu.STL; visual mesh filename=package://stretch_description/meshes/base_imu.STL
- added link link_grasp_center
- link base_link: mass 1.1912 -> 17.384389; geometry collision mesh filename=package://stretch_description/meshes/base_link.STL; visual mesh filename=package://stretch_description/meshes/base_link.STL
- link camera_link: geometry collision box size=0.02505 0.09 0.025; visual mesh filename=package://realsense2_description/meshes/d435.dae
- link caster_link: geometry collision sphere radius=0.032; visual mesh filename=package://stretch_description/meshes/omni_wheel_m.STL
- link laser: mass 0.0749979022894495 -> 0.216007; geometry collision mesh filename=package://stretch_description/meshes/laser.STL; visual mesh filename=package://stretch_description/meshes/laser.STL
- link link_arm_l0: mass 0.085003260946398 -> 0.427734; geometry collision mesh filename=package://stretch_description/meshes/link_arm_l0.STL; visual mesh filename=package://stretch_description/meshes/link_arm_l0.STL
- link link_arm_l1: mass 0.051382 -> 0.113658; geometry collision mesh filename=package://stretch_description/meshes/link_arm_l1.STL; visual mesh filename=package://stretch_description/meshes/link_arm_l1.STL
- link link_arm_l2: mass 0.0571386353275368 -> 0.130565; geometry collision mesh filename=package://stretch_description/meshes/link_arm_l2.STL; visual mesh filename=package://stretch_description/meshes/link_arm_l2.STL
- link link_arm_l3: mass 0.0628927381893134 -> 0.146817; geometry collision mesh filename=package://stretch_description/meshes/link_arm_l3.STL; visual mesh filename=package://stretch_description/meshes/link_arm_l3.STL
- link link_arm_l4: mass 0.068095 -> 0.235626; geometry collision mesh filename=package://stretch_description/meshes/link_arm_l4.STL; visual mesh filename=package://stretch_description/meshes/link_arm_l4.STL
- link link_aruco_inner_wrist: geometry collision mesh filename=package://stretch_description/meshes/link_aruco_inner_wrist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; visual mesh filename=package://stretch_description/meshes/link_aruco_inner_wrist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
- link link_aruco_left_base: geometry collision mesh filename=package://stretch_description/meshes/link_aruco_left_base.S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; visual mesh filename=package://stretch_description/meshes/link_aruco_left_base.S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
- link link_aruco_right_base: geometry collision mesh filename=package://stretch_description/meshes/link_aruco_right_base.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; visual mesh filename=package://stretch_description/meshes/link_aruco_right_base.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
- link link_aruco_shoulder: geometry collision mesh filename=package://stretch_description/meshes/link_aruco_shoulder.STL; visual mesh filename=package://stretch_description/meshes/link_aruco_shoulder.STL
- link link_aruco_top_wrist: geometry collision mesh filename=package://stretch_description/meshes/link_aruco_top_wrist.S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; visual mesh filename=package://stretch_description/meshes/link_aruco_top_wrist.S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
- link link_gripper_finger_left: mass 0.0476207785199479 -> 0.06; geometry collision mesh filename=package://stretch_description/meshes/link_gripper_finger_le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; visual mesh filename=package://stretch_description/meshes/link_gripper_finger_le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
- link link_gripper_finger_right: mass 0.047621 -> 0.06; geometry collision mesh filename=package://stretch_description/meshes/link_gripper_finger_ri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; visual mesh filename=package://stretch_description/meshes/link_gripper_finger_ri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
- link link_gripper_fingertip_left: mass 0.00382160686584851 -> 0.003822; geometry collision mesh filename=package://stretch_description/meshes/link_gripper_fingertip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; visual mesh filename=package://stretch_description/meshes/link_gripper_fingertip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
- link link_gripper_fingertip_right: mass 0.00382160881468841 -> 0.003822; geometry collision mesh filename=package://stretch_description/meshes/link_gripper_fingertip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; visual mesh filename=package://stretch_description/meshes/link_gripper_fingertip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
- link link_head: mass 0.133027236718691 -> 0.681871; geometry collision mesh filename=package://stretch_description/meshes/link_head.STL; visual mesh filename=package://stretch_description/meshes/link_head.STL
- link link_head_pan: mass 0.0273764496535409 -> 0.062462; geometry collision mesh filename=package://stretch_description/meshes/link_head_pan.STL; visual mesh filename=package://stretch_description/meshes/link_head_pan.STL
- link link_head_tilt: mass 0.090217113313934 -> 0.283548; geometry collision mesh filename=package://stretch_description/meshes/link_head_tilt.STL; visual mesh filename=package://stretch_description/meshes/link_head_tilt.STL
- link link_left_wheel: mass 0.0042721 -> 0.20773; geometry collision mesh filename=package://stretch_description/meshes/link_left_wheel.STL; visual mesh filename=package://stretch_description/meshes/link_left_wheel.STL
- link link_lift: mass 0.27218 -> 1.987167; geometry collision mesh filename=package://stretch_description/meshes/link_lift.STL; visual mesh filename=package://stretch_description/meshes/link_lift.STL
- link link_mast: mass 1.8285 -> 1.764017; geometry collision mesh filename=package://stretch_description/meshes/link_mast.STL; visual mesh filename=package://stretch_description/meshes/link_mast.STL
- link link_right_wheel: mass 0.0042721 -> 0.20773; geometry collision mesh filename=package://stretch_description/meshes/link_right_wheel.STL; visual mesh filename=package://stretch_description/meshes/link_right_wheel.STL
- link link_straight_gripper: mass 0.0496384234458284 -> 0.147853; geometry collision mesh filename=package://stretch_description/meshes/link_straight_gripper.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; visual mesh filename=package://stretch_description/meshes/link_straight_gripper.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
- link link_wrist_pitch: mass 0.0701267146295583 -> 0.208129; geometry collision mesh filename=package://stretch_description/meshes/link_wrist_pitch.STL; visual mesh filename=package://stretch_description/meshes/link_wrist_pitch.STL
- link link_wrist_roll: mass 0.00585666394358811 -> 0.01528; geometry collision mesh filename=package://stretch_description/meshes/link_wrist_roll.STL; visual mesh filename=package://stretch_description/meshes/link_wrist_roll.STL
- link link_wrist_yaw: mass 0.0404746907425003 -> 0.054422; geometry collision mesh filename=package://stretch_description/meshes/link_wrist_yaw.STL; visual mesh filename=package://stretch_description/meshes/link_wrist_yaw.STL
- link link_wrist_yaw_bottom: mass 0.0988906816399982 -> 0.24284; geometry collision mesh filename=package://stretch_description/meshes/link_wrist_yaw_bottom.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; visual mesh filename=package://stretch_description/meshes/link_wrist_yaw_bottom.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
- link respeaker_base: mass 0.015643 -> 0.025175; geometry collision mesh filename=package://stretch_description/meshes/respeaker_base.STL; visual mesh filename=package://stretch_description/meshes/respeaker_base.STL
Joints:
- removed joint base_theta_joint
- removed joint base_x_joint
- removed joint base_y_joint
- added joint joint_base_imu: type fixed, parent base_link, child base_imu, origin xyz=-0.12838 0.0031592 0.1474 rpy=-3.1416 0.0 -1.5708, axis 0.0 0.0 0.0
- added joint joint_grasp_center: type fixed, parent link_straight_gripper, child link_grasp_center, origin xyz=0.0 0.0 0.23 rpy=-1.5707963267949 -1.5707963267949 0.0
- joint camera_joint: origin xyz=0.02802960503838624 -0.007608222297947431 0.018218494141479257 rpy=0.010658876360659654 -0.0022761048951753793 0.018675317090921212 -> xyz=0.02594509431127206 -0.009367287969076725 0.01787783107637637 rpy=0.017722981056775697 -0.0025107850545702526 0.032908414619659106
- joint joint_arm_l4: origin xyz=-0.25956015433181046 -0.0059261537843136765 -0.005557384627505743 rpy=1.5619286973774569 -0.006924580188019336 -1.575847166561953 -> xyz=-0.2577874700535916 -0.006741141968681925 0.004433978643577055 rpy=1.5926663544429687 0.036934383992214714 -1.554250155712327
- joint joint_head_pan: origin xyz=0.1284513021260868 0.07637128403435504 0.00023722543808071166 rpy=-0.013467967166369273 0.005690738105448956 1.6024957766579377 -> xyz=0.1324676880114166 0.07690307833191154 -0.008108842131907289 rpy=0.0035478588117889252 0.0158595575891618 1.5221917799002653
- joint joint_head_tilt: origin xyz=0.0032337815907659225 0.030910701770693223 -0.04783143162927699 rpy=1.5763332066189244 -0.029319157204454882 -0.005080558641851002 -> xyz=0.003831886692638425 0.028708440719587294 -0.045015975487188595 rpy=1.5815726358488218 0.0067993179483869515 0.0023152040737468636
- joint joint_mast: origin xyz=-0.07174416574437388 0.13780491000396983 0.03663931715774088 rpy=1.5780076046568878 0.016499709009588637 -0.007971437955302632 -> xyz=-0.07218435917539559 0.13510471622868134 0.03664565218339203 rpy=1.5686223488284634 -0.004600755654868616 0.0032835266112827225
